Commit message: feat(webots): vendor TIAGo visuals via pinned local meshes
Ship URDF overlays, license notes, and a vendor script while keeping generated mesh and texture trees out of Git.

Assisted-by: Cursor:Composer

File: examples/webots/sim/ros_ws/src/eaios_webots/resource/tiago_full_webots.urdf (robot description, URDF)
Before this commit: robot Tiago Webots, 39 links, 38 joints
Links:
- added link arm_1_link, mass 1.563428; collision mesh filename=meshes/stl/tiago_description__meshes__arm__arm_1_collision.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 scale=1 1 1; visual mesh filename=meshes/stl/tiago_description__meshes__arm__arm_1.stl scale=1 1 1
- added link arm_2_link, mass 1.800397; collision mesh filename=meshes/stl/tiago_description__meshes__arm__arm_2_collision.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 scale=1 1 1; visual mesh filename=meshes/stl/tiago_description__meshes__arm__arm_2.stl scale=1 1 1
- added link arm_3_link, mass 1.8; collision mesh filename=meshes/stl/tiago_description__meshes__arm__arm_3_collision.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 scale=1 1 1; visual mesh filename=meshes/stl/tiago_description__meshes__arm__arm_3.stl scale=1 1 1
- added link arm_4_link, mass 1.432697; collision mesh filename=meshes/stl/tiago_description__meshes__arm__arm_4_collision.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 scale=1 1 1; visual mesh filename=meshes/stl/tiago_description__meshes__arm__arm_4.stl scale=1 1 1
- added link arm_5_link, mass 0.9359143689; collision mesh filename=meshes/stl/tiago_description__meshes__arm__arm_5_collision-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 scale=1 1 1; visual mesh filename=meshes/stl/tiago_description__meshes__arm__arm_5-wrist-2017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 scale=1 1 1
- added link arm_6_link, mass 0.30275767222; collision mesh filename=meshes/stl/tiago_description__meshes__arm__arm_6_collision-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 scale=1 1 1; visual mesh filename=meshes/stl/tiago_description__meshes__arm__arm_6-wrist-2017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 scale=1 1 1
- added link arm_7_link, mass 0.100
- added link arm_tool_link, mass 0.1; collision cylinder length=0.005 radius=0.005; visual cylinder length=0.005 radius=0.005
- added link gripper_grasping_frame, mass 0.1
- added link gripper_left_finger_link, mass 0.107001; collision box size=0.01 0.05 0.11; visual mesh filename=meshes/stl/pal_gripper_description__meshes__gripper_finger_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
- added link gripper_link, mass 0.602660; collision mesh filename=meshes/stl/pal_gripper_description__meshes__gripper_link_co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; visual mesh filename=meshes/stl/pal_gripper_description__meshes__gripper_link.stl
- added link gripper_right_finger_link, mass 0.107001; collision box size=0.01 0.05 0.11; visual mesh filename=meshes/stl/pal_gripper_description__meshes__gripper_finger_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 scale=-1 -1 1
- added link gripper_tool_link
- added link wrist_ft_link, mass 0.095000; collision cylinder length=0.0157 radius=0.0225; visual cylinder length=0.0157 radius=0.0225
- added link wrist_ft_tool_link, mass 0.1; collision cylinder length=0.00975 radius=0.025; visual cylinder length=0.00975 radius=0.025
Joints:
- added joint arm_1_joint: type revolute, parent torso_lift_link, child arm_1_link, origin xyz=0.15505 0.014 -0.151 rpy=0 0 -1.5707963267948966, axis 0 0 1, limit lower=0.0 upper=2.748893571891069 effort=43.0 velocity=1.95
- added joint arm_2_joint: type revolute, parent arm_1_link, child arm_2_link, origin xyz=0.125 0.0195 -0.031 rpy=1.5707963267948966 0.0 0.0, axis 0 0 1, limit lower=-1.5707963267948966 upper=1.090830782496456 effort=43.0 velocity=1.95
- added joint arm_3_joint: type revolute, parent arm_2_link, child arm_3_link, origin xyz=0.0895 0.0 0.0015 rpy=-1.5707963267948966 0.0 1.5707963267948966, axis 0 0 1, limit lower=-3.5342917352885173 upper=1.5707963267948966 effort=26 velocity=2.35
- added joint arm_4_joint: type revolute, parent arm_3_link, child arm_4_link, origin xyz=-0.02 -0.027 -0.222 rpy=-1.5707963267948966 -1.5707963267948966 0.0, axis 0 0 1, limit lower=-0.39269908169872414 upper=2.356194490192345 effort=26 velocity=2.35
- added joint arm_5_joint: type revolute, parent arm_4_link, child arm_5_link, origin xyz=-0.162 0.02 0.027 rpy=1.5707963267948966 -1.5707963267948966 -1.5707963267948966, axis 0 0 1, limit lower=-2.0943951023931953 upper=2.0943951023931953 effort=3 velocity=1.95
- added joint arm_6_joint: type revolute, parent arm_5_link, child arm_6_link, origin xyz=0 0 0.15 rpy=0.0 -1.5707963267948966 -1.5707963267948966, axis 0 0 1, limit lower=-1.413716694115407 upper=1.413716694115407 effort=6.6 velocity=1.76
- added joint arm_7_joint: type revolute, parent arm_6_link, child arm_7_link, origin xyz=0 0 0 rpy=1.5707963267948966 0.0 1.5707963267948966, axis 0 0 1, limit lower=-2.0943951023931953 upper=2.0943951023931953 effort=6.6 velocity=1.76
- added joint arm_tool_joint: type fixed, parent arm_7_link, child arm_tool_link, origin xyz=0 0 0.051875 rpy=1.5707963267948966 -1.5707963267948966 3.141592653589793
- added joint gripper_grasping_frame_joint: type fixed, parent gripper_link, child gripper_grasping_frame, origin xyz=0 0 -0.13 rpy=-1.5708 1.5708 0
- added joint gripper_joint: type fixed, parent wrist_ft_tool_link, child gripper_link, origin xyz=0 0 0 rpy=1.5707963267948966 1.5707963267948966 -1.5707963267948966, axis 0 0 0
- added joint gripper_left_finger_joint: type prismatic, parent gripper_link, child gripper_left_finger_link, origin xyz=0 0 -0.01 rpy=0 0 0, axis -1 0 0, limit lower=0.0 upper=0.045 effort=16 velocity=0.05
- added joint gripper_right_finger_joint: type prismatic, parent gripper_link, child gripper_right_finger_link, origin xyz=0 0 -0.01 rpy=0 0 0, axis 1 0 0, limit lower=0.0 upper=0.045 effort=16 velocity=0.05
- added joint gripper_tool_joint: type fixed, parent wrist_ft_tool_link, child gripper_tool_link, origin xyz=0 0 0 rpy=1.5707963267948966 1.5707963267948966 -1.5707963267948966, axis 0 0 0
- added joint wrist_ft_joint: type fixed, parent arm_tool_link, child wrist_ft_link, origin xyz=0 0 0 rpy=0 1.5707963267948966 0
- added joint wrist_tool_joint: type fixed, parent wrist_ft_link, child wrist_ft_tool_link, origin xyz=0 0 0.0112 rpy=0 -1.5707963267948966 0
